Commit message: fix launch configuration and urdf file for real robot setup

File: robotiq_85_description/urdf/robotiq_85_gripper.xacro (robot description, xacro)
@@ -7,33 +7,7 @@
         </plugin>
     </gazebo>
-    <link name="world"/>
-    <joint name="world_fixed" type="fixed">
+    <link name="gripper_root"/>
+    <xacro:robotiq_85_gripper prefix="" parent="gripper_root" >
         <origin xyz="0 0 0" rpy="0 0 0"/>
-        <parent link="world"/>
-        <child link="gripper_root_link"/>
-    </joint>
-    <link name="gripper_root_link">
-        <visual>
-            <origin xyz="0 0 0.5" rpy="0 0 0"/>
-            <geometry>
-                <box size="0.1 0.1 1.0"/>
-            </geometry>
-        </visual>
-        <collision>
-            <origin xyz="0 0 0.5" rpy="0 0 0"/>
-            <geometry>
-                <box size="0.1 0.1 1.0"/>
-            </geometry>
-        </collision>
-        <inertial>
-            <mass value="1e2" />
-            <origin xyz="0.0 0.0 0.0" />
-            <inertia ixx = "0.000001" ixy = "0.000000" ixz = "0.000000"
-                     iyx = "0.000000" iyy = "0.000001" iyz = "0.000000"
-                     izx = "0.000000" izy = "0.000000" izz = "0.000001" />
-        </inertial>
-    </link>
-    <xacro:robotiq_85_gripper prefix="" parent="gripper_root_link" >
-        <origin xyz="0.05 0 0.85" rpy="0 0 0"/>
     </xacro:robotiq_85_gripper>
 </robot>
